Commit message: controller, velodyne updated

File: urdf/hunter_with_one_box.urdf.xacro (robot description, xacro)
@@ -3,4 +3,8 @@
   <!-- Include the original hunter description -->
   <xacro:include filename="$(find scv_robot_gazebo)/robots/hunter_robot/hunter_description/description/robot_core.xacro" />
+  <!-- Include ROS2 control for Hunter robot -->
+  <xacro:include filename="$(find scv_robot_gazebo)/robots/hunter_robot/hunter_description/description/ros2_control.xacro" />
+  <!-- Include VLP-32C sensor (local version with correct mesh path) -->
+  <xacro:include filename="$(find scv_robot_gazebo)/urdf/velodyne_vlp32c.urdf.xacro" />
   <!-- Add front box with DAE mesh (Hunter style) -->
   <link name="front_box">
@@ -59,3 +63,7 @@
     <origin xyz="-0.0865 0 0.093" rpy="0 0 0"/>
   </joint>
+  <!-- VLP-32C Lidar on front box (same position as SCV) -->
+  <xacro:VLP-32C parent="front_box" name="velodyne" topic="/velodyne_points">
+    <origin xyz="-0.036 0 0.162" rpy="0 0 0"/>
+  </xacro:VLP-32C>
 </robot>

Commit message: GPS, IMU 센서 추가 - 다만 GPS 센서의 경우 원점(0, 0, 0)을 기준으로 하므로 추가 설정 필요해 보임

File: urdf/hunter_with_one_box.urdf.xacro (robot description, xacro)
@@ -67,3 +67,164 @@
     <origin xyz="-0.036 0 0.162" rpy="0 0 0"/>
   </xacro:VLP-32C>
+  <!-- GNSS antenna on back box -->
+  <link name="gnss_antenna">
+    <visual>
+      <origin xyz="0 0 0" rpy="1.5708 0 0"/>
+      <geometry>
+        <mesh filename="file://$(find scv_robot_gazebo)/meshes/GNSS_antenna.stl" scale="0.001 0.001 0.001"/>
+      </geometry>
+      <material name="white">
+        <color rgba="0.9 0.9 0.9 1.0"/>
+      </material>
+    </visual>
+    <collision>
+      <origin xyz="0 0 0" rpy="0 0 0"/>
+      <geometry>
+        <cylinder radius="0.02" length="0.05"/>
+      </geometry>
+    </collision>
+    <inertial>
+      <origin xyz="0 0 0" rpy="0 0 0"/>
+      <mass value="0.1"/>
+      <inertia ixx="0.001" ixy="0.0" ixz="0.0" iyy="0.001" iyz="0.0" izz="0.001"/>
+    </inertial>
+  </link>
+  <joint name="gnss_antenna_joint" type="fixed">
+    <parent link="back_box"/>
+    <child link="gnss_antenna"/>
+    <origin xyz="0 0 0.15" rpy="0 0 0"/>
+  </joint>
+  <!-- GPS sensor for Gazebo -->
+  <gazebo reference="gnss_antenna">
+    <sensor name="gps_sensor" type="gps">
+      <pose>0 0 0 0 0 0</pose>
+      <always_on>1</always_on>
+      <update_rate>10.0</update_rate>
+      <gps>
+        <position_sensing>
+          <horizontal>
+            <noise type="gaussian">
+              <mean>0.0</mean>
+              <stddev>0.1</stddev>
+            </noise>
+          </horizontal>
+          <vertical>
+            <noise type="gaussian">
+              <mean>0.0</mean>
+              <stddev>0.1</stddev>
+            </noise>
+          </vertical>
+        </position_sensing>
+        <velocity_sensing>
+          <horizontal>
+            <noise type="gaussian">
+              <mean>0.0</mean>
+              <stddev>0.1</stddev>
+            </noise>
+          </horizontal>
+          <vertical>
+            <noise type="gaussian">
+              <mean>0.0</mean>
+              <stddev>0.1</stddev>
+            </noise>
+          </vertical>
+        </velocity_sensing>
+      </gps>
+      <plugin name="gps_plugin" filename="libgazebo_ros_gps_sensor.so">
+        <ros>
+          <namespace>/</namespace>
+          <remapping>~/out:=gps/fix</remapping>
+        </ros>
+        <frame_name>gnss_antenna</frame_name>
+        <reference_latitude>37.5665</reference_latitude>
+        <reference_longitude>126.9780</reference_longitude>
+        <reference_altitude>50.0</reference_altitude>
+      </plugin>
+    </sensor>
+  </gazebo>
+  <!-- IMU sensor link -->
+  <link name="imu_link">
+    <visual>
+      <origin xyz="0 0 0" rpy="0 0 0"/>
+      <geometry>
+        <box size="0.02 0.02 0.01"/>
+      </geometry>
+      <material name="black">
+        <color rgba="0.1 0.1 0.1 1.0"/>
+      </material>
+    </visual>
+    <collision>
+      <origin xyz="0 0 0" rpy="0 0 0"/>
+      <geometry>
+        <box size="0.02 0.02 0.01"/>
+      </geometry>
+    </collision>
+    <inertial>
+      <origin xyz="0 0 0" rpy="0 0 0"/>
+      <mass value="0.01"/>
+      <inertia ixx="0.0001" ixy="0.0" ixz="0.0" iyy="0.0001" iyz="0.0" izz="0.0001"/>
+    </inertial>
+  </link>
+  <joint name="imu_joint" type="fixed">
+    <parent link="chassis"/>
+    <child link="imu_link"/>
+    <origin xyz="0 0 0.05" rpy="0 0 0"/>
+  </joint>
+  <!-- IMU sensor for Gazebo -->
+  <gazebo reference="imu_link">
+    <sensor name="imu_sensor" type="imu">
+      <pose>0 0 0 0 0 0</pose>
+      <always_on>1</always_on>
+      <update_rate>100.0</update_rate>
+      <imu>
+        <angular_velocity>
+          <x>
+            <noise type="gaussian">
+              <mean>0.0</mean>
+              <stddev>0.02</stddev>
+            </noise>
+          </x>
+          <y>
+            <noise type="gaussian">
+              <mean>0.0</mean>
+              <stddev>0.02</stddev>
+            </noise>
+          </y>
+          <z>
+            <noise type="gaussian">
+              <mean>0.0</mean>
+              <stddev>0.02</stddev>
+            </noise>
+          </z>
+        </angular_velocity>
+        <linear_acceleration>
+          <x>
+            <noise type="gaussian">
+              <mean>0.0</mean>
+              <stddev>0.1</stddev>
+            </noise>
+          </x>
+          <y>
+            <noise type="gaussian">
+              <mean>0.0</mean>
+              <stddev>0.1</stddev>
+            </noise>
+          </y>
+          <z>
+            <noise type="gaussian">
+              <mean>0.0</mean>
+              <stddev>0.1</stddev>
+            </noise>
+          </z>
+        </linear_acceleration>
+      </imu>
+      <plugin name="imu_plugin" filename="libgazebo_ros_imu_sensor.so">
+        <ros>
+          <namespace>/</namespace>
+          <remapping>~/out:=imu/data</remapping>
+        </ros>
+        <frame_name>imu_link</frame_name>
+      </plugin>
+    </sensor>
+  </gazebo>
 </robot>

File: urdf/velodyne_vlp32c.urdf.xacro (robot description, xacro)
@@ -15,5 +15,5 @@
       </inertial>
       <visual>
-        <origin xyz="0 0 0" rpy="0 0 0"/>
+        <origin xyz="0 0 0" rpy="1.5708 0 0"/>
         <geometry>
           <mesh filename="file://$(find scv_robot_gazebo)/meshes/VLP-32C.stl" scale="0.001 0.001 0.001"/>

Commit message: GPS 기준좌표 수정 진행중

File: urdf/hunter_with_one_box.urdf.xacro (robot description, xacro)
@@ -1,4 +1,11 @@
 <?xml version="1.0"?>
 <robot name="hunter_with_one_box" xmlns:xacro="http://www.ros.org/wiki/xacro">
+  <!-- GPS reference coordinates parameters -->
+  <xacro:arg name="gps_latitude" default="37.5665"/>
+  <xacro:arg name="gps_longitude" default="126.9780"/>
+  <xacro:arg name="gps_altitude" default="50.0"/>
+  <xacro:property name="gps_ref_lat" value="$(arg gps_latitude)"/>
+  <xacro:property name="gps_ref_lon" value="$(arg gps_longitude)"/>
+  <xacro:property name="gps_ref_alt" value="$(arg gps_altitude)"/>
   <!-- Include the original hunter description -->
   <xacro:include filename="$(find scv_robot_gazebo)/robots/hunter_robot/hunter_description/description/robot_core.xacro" />
@@ -137,7 +144,7 @@
         </ros>
         <frame_name>gnss_antenna</frame_name>
-        <reference_latitude>37.5665</reference_latitude>
-        <reference_longitude>126.9780</reference_longitude>
-        <reference_altitude>50.0</reference_altitude>
+        <reference_latitude>${gps_ref_lat}</reference_latitude>
+        <reference_longitude>${gps_ref_lon}</reference_longitude>
+        <reference_altitude>${gps_ref_alt}</reference_altitude>
       </plugin>
     </sensor>
